File: pcb/cpu.kicad_sch (KiCad schematic)
At the start: 13 parts, among them SW1 T1B2QR, U1 F1C200s, Y1 24Mhz

Commit message: Added last minor patches like ideal diode on PCB, added backplate
Connections:
- net GND: no longer U1.2 (HPCOMFB), U1.3 (HPCOM)
- new net HPCOM: U1.2 (HPCOMFB), U1.3 (HPCOM)
Changed lines of the file:
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@@
+		)
+	)
+	(global_label "HPCOM"
+		(shape input)
+		(at 203.2 127 0)
+		(fields_autoplaced yes)
+		(effects
+			(font
+				(size 1.27 1.27)
+			)
+			(justify left)
+		)
+		(property "Intersheetrefs" "${INTERSHEET_REFS}"
+			(at 212.8376 127 0)
+			(effects
+				(font
+					(size 1.27 1.27)
+				)
+				(justify left)
+				(hide yes)
+			)
 		)
 	)
@@
 					(unit 1)
 				)
-			)
-		)
-	)
-	(symbol
-		(lib_id "power:GND")
-		(at 203.2 127 90)
-		(unit 1)
-		(exclude_from_sim no)
-		(in_bom yes)
-		(on_board yes)
-		(dnp no)
-		(fields_autoplaced yes)
-		(property "Reference" "#PWR01"
-			(at 209.55 127 0)
-			(effects
-				(font
-					(size 1.27 1.27)
-				)
-				(hide yes)
-			)
-		)
-		(property "Value" "GND"
-			(at 207.01 127.6349 90)
-			(effects
-				(font
-					(size 1.27 1.27)
-				)
-				(justify right)
-			)
-		)
-		(property "Footprint" ""
-			(at 203.2 127 0)
-			(effects
-				(font
-					(size 1.27 1.27)
-				)
-				(hide yes)
-			)
-		)
-		(property "Datasheet" ""
-			(at 203.2 127 0)
-			(effects
-				(font
-					(size 1.27 1.27)
-				)
-				(hide yes)
-			)
-		)
-		(property "Description" ""
-			(at 203.2 127 0)
-			(effects
-				(font
-					(size 1.27 1.27)
-				)
-				(hide yes)
-			)
-		)
-		(pin "1"
-		)
-		(instances
-			(project "minidisc"
-				(path "/521fcede-69d7-4f6d-a594-609fca379ec3/0047e17d-33b3-4049-9b95-9a904173d4c1"
-					(reference "#PWR01")
-					(unit 1)
-				)
