File: pcb/minidisc.kicad_pcb (KiCad board)
At the start: 4 copper layers, 96 x 78 mm, 142 parts, among them J1 Conn_01x02, J4 Conn_01x20, J5 SATA_USB, J6 CPU_USB, Q1 AO3400_C181090, Q2 AO3401A, SW1 T1B2QR, SW2 PLAY, SW3 SPVS410100, SW4 STOP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

Commit message: Added last minor patches like ideal diode on PCB, added backplate
Parts:
- removed D1: 1N5819, Diode_SMD:D_SOD-123
- added Q3: DMG2305UX-7, lcsc:SOT-23-3_L2.9-W1.3-P1.90-LS2.4-BR, F.Cu at (149.2, 63.1)
- added Q4: DMMT5401-7-F, lcsc:SOT-23-6_L2.9-W1.6-P0.95-LS2.8-BR, F.Cu at (150.5, 38.9)
- added R23: 47k 1%, Resistor_SMD:R_0402_1005Metric, F.Cu at (158.8, 42.0)
- added R26: 47k 1%, Resistor_SMD:R_0402_1005Metric, F.Cu at (158.8, 44.0)
- R4: value 1.1K -> 4.7k
Connections:
- Audio1 pad 1: GND -> HPCOM
- C10 pad 1: /Power/+5V_ALWAYS -> +5V_ALWAYS
- C7 pad 1: /Power/+5V_ALWAYS -> +5V_ALWAYS
- D4 pad 1: /Power/+5V_ALWAYS -> +5V_ALWAYS
- Q2 pad 2: /Power/+5V_ALWAYS -> +5V_ALWAYS
- R40 pad 1: BTPWR -> Net-(R40-Pad1)
- R40 pad 2: GND -> BTPWR
- R41 pad 1: +5V -> +5V_ALWAYS
- R42 pad 1: /Power/+5V_ALWAYS -> +5V_ALWAYS
- SW9 pad 2: BTPWR -> Net-(R40-Pad1)
- U1 pad 2: GND -> HPCOM
- U1 pad 3: GND -> HPCOM
- U2 pad 1: /Power/+5V_ALWAYS -> +5V_ALWAYS
Routing:
- net +5V_ALWAYS: track 0.00 -> 158.8 mm, vias 0 -> 3
- net /Power/+5V_ALWAYS: track 155.8 -> 0.00 mm, vias 2 -> 0
- net HPCOM: track 0.00 -> 27.2 mm, vias 0 -> 3
- net GND: track 175.7 -> 169.0 mm, vias 119 -> 115
- net +5V: track 277.6 -> 272.9 mm, vias 14 -> 12
- net +5VD: track 85.3 -> 82.1 mm
- net Net-(R40-Pad1): track 0.00 -> 2.30 mm
- net BTPWR: track 138.4 -> 137.0 mm
